File: stm32 clone/stm32 clone.kicad_sch (KiCad schematic)
At the start: 10 parts, among them U1 STM32G030C6T6, Y1 8 MHz, Y2 32.768 KHz

Commit message: reset circuit, debug
Parts:
- added J1: DEBUG, Package_DFN_QFN:QFN-24-1EP_4x4mm_P0.5mm_EP2.6x2.6mm, symbol Connector_Generic:Conn_01x05
- C1, C3: value 100n -> 100nF; footprint Package_QFP:LQFP-48_7x7mm_P0.5mm -> Capacitor_SMD:C_0805_2012Metric_Pad1.18x1.45mm_HandSolder
- C2: value 4.7u -> 4.7uF; footprint Package_QFP:LQFP-48_7x7mm_P0.5mm -> Capacitor_SMD:C_0805_2012Metric_Pad1.18x1.45mm_HandSolder
- C4, C5: value 22p -> 22pF; footprint Package_QFP:LQFP-48_7x7mm_P0.5mm -> Capacitor_SMD:C_0805_2012Metric_Pad1.18x1.45mm_HandSolder
- C6, C7: value 18p -> 18pF; footprint Package_QFP:LQFP-48_7x7mm_P0.5mm -> Capacitor_SMD:C_0805_2012Metric_Pad1.18x1.45mm_HandSolder
Connections:
- net +3.3V: now also J1.5 (Pin_5)
- net GND: now also J1.3 (Pin_3)
- net NRST: now reaches U1.10 (NRST)
- net NRST: now also J1.1 (Pin_1)
- net SWDIO: now reaches U1.35 (PA13)
- net SWDIO: now also J1.2 (Pin_2)
- net SWCLK: now reaches U1.36 (PA14-BOOT0)
- net SWCLK: now also J1.4 (Pin_4)

Commit message: cubeide config
Parts:
- added C8: 0.1uF, Package_SO:SOIC-8_3.9x4.9mm_P1.27mm, symbol Device:C
- added SW1: RST, Button_Switch_THT:SW_PUSH_6mm_2pin, symbol Switch:SW_Push
Connections:
- net GND: now also C8.2, SW1.2
- net NRST: now also C8.1, SW1.1
Other:
- note added: "Reset circuit"
