File: stm32 clone/stm32 clone.kicad_sch (KiCad schematic)
At the start: 13 parts, among them J1 DEBUG, SW1 RST, U1 STM32G030C6T6, Y1 8 MHz, Y2 32.768 KHz

Commit message: usb c started
Parts:
- added C9: 10uF, symbol Device:C
- added D1: D_Schottky, symbol Device:D_Schottky
- added J2: USB_C_Receptacle_USB2.0_16P, Connector_USB:USB_C_Receptacle_GCT_USB4105-xx-A_16P_TopMnt_Horizontal, symbol Connector:USB_C_Receptacle_USB2.0_16P
- added R1, R2: 5k1, symbol Device:R
Connections:
- net GND: now also C9.2, J2.A1 (GND), J2.A12 (GND), J2.B1 (GND), J2.B12 (GND), J2.SH (SHIELD)
- new net: D1.2 (A), J2.A4 (VBUS), J2.A9 (VBUS), J2.B4 (VBUS), J2.B9 (VBUS)
- new net +5V: C9.1, D1.1 (K)
- no-connect marks 0 -> 6

Commit message: comments, usb c
Parts:
- C8: footprint Package_SO:SOIC-8_3.9x4.9mm_P1.27mm -> Capacitor_SMD:C_0805_2012Metric_Pad1.18x1.45mm_HandSolder
- C9: footprint (none) -> Capacitor_SMD:C_0805_2012Metric_Pad1.18x1.45mm_HandSolder
- D1: value D_Schottky -> 1N5819; footprint (none) -> Diode_THT:D_DO-15_P12.70mm_Horizontal; MAN (none) -> 1N5819; TME (none) -> 1N5819-DIO; URL (none) -> https://www.tme.eu/pl/details/1n5819-dio/diody-schottky-tht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
- R1, R2: footprint (none) -> Resistor_SMD:R_0805_2012Metric_Pad1.20x1.40mm_HandSolder
Connections:
- net GND: now also R1.2, R2.2
- net at R1.1: now also J2.B5 (CC2)
- net at R2.1: now also J2.A5 (CC1)
Changed lines of the file:
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@@
 		(comment 1 "TODO: add blink in nice spot in pcb design phase")
 		(comment 2 "TODO: add usr button")
+		(comment 3 "TODO: TVS diode")
+		(comment 4 "TODO: LDO to 3.3")
 	)
 	(rectangle
@@
 	)
 	(junction
+		(at 67.31 59.69)
+		(diameter 0)
+		(color 0 0 0 0)
+	)
+	(junction
 		(at 44.45 107.95)
 		(diameter 0)
@@
 	)
 	(junction
+		(at 59.69 59.69)
+		(diameter 0)
+		(color 0 0 0 0)
+	)
+	(junction
 		(at 48.26 144.78)
 		(diameter 0)
@@
 	(wire
 		(pts
+			(xy 59.69 49.53) (xy 59.69 59.69)
+		)
+		(stroke
+			(width 0)
+			(type default)
+		)
+	)
+	(wire
+		(pts
 			(xy 250.19 80.01) (xy 266.7 80.01)
 		)
@@
 	(wire
 		(pts
+			(xy 52.07 59.69) (xy 59.69 59.69)
+		)
+		(stroke
+			(width 0)
+			(type default)
+		)
+	)
+	(wire
+		(pts
+			(xy 59.69 33.02) (xy 59.69 41.91)
+		)
+		(stroke
+			(width 0)
+			(type default)
+		)
+	)
+	(wire
+		(pts
 			(xy 160.02 81.28) (xy 177.8 81.28)
 		)
@@
 	(wire
 		(pts
+			(xy 46.99 35.56) (xy 52.07 35.56)
+		)
+		(stroke
+			(width 0)
+			(type default)
+		)
+	)
+	(wire
+		(pts
 			(xy 25.4 144.78) (xy 25.4 154.94)
 		)
@@
 	(wire
 		(pts
+			(xy 59.69 59.69) (xy 67.31 59.69)
+		)
+		(stroke
+			(width 0)
+			(type default)
+		)
+	)
+	(wire
+		(pts
 			(xy 224.79 30.48) (xy 234.95 30.48)
 		)
@@
 	(wire
 		(pts
+			(xy 52.07 35.56) (xy 52.07 41.91)
+		)
+		(stroke
+			(width 0)
+			(type default)
+		)
+	)
+	(wire
+		(pts
 			(xy 30.48 154.94) (xy 25.4 154.94)
 		)
@@
 	(wire
 		(pts
+			(xy 52.07 49.53) (xy 52.07 59.69)
+		)
+		(stroke
+			(width 0)
+			(type default)
+		)
+	)
+	(wire
+		(pts
+			(xy 67.31 59.69) (xy 67.31 63.5)
+		)
+		(stroke
+			(width 0)
+			(type default)
+		)
+	)
+	(wire
+		(pts
 			(xy 107.95 91.44) (xy 124.46 91.44)
 		)
@@
 	(wire
 		(pts
-			(xy 67.31 43.18) (xy 67.31 63.5)
+			(xy 67.31 43.18) (xy 67.31 59.69)
 		)
 		(stroke
@@
 	(wire
 		(pts
+			(xy 46.99 33.02) (xy 59.69 33.02)
+		)
+		(stroke
+			(width 0)
+			(type default)
+		)
+	)
+	(wire
+		(pts
 			(xy 107.95 66.04) (xy 124.46 66.04)
 		)
@@
 			)
 		)
-		(property "Footprint" ""
+		(property "Footprint" "Resistor_SMD:R_0805_2012Metric_Pad1.20x1.40mm_HandSolder"
 			(at 50.292 45.72 90)
 			(hide yes)
@@
 			)
 		)
-		(property "Footprint" ""
+		(property "Footprint" "Resistor_SMD:R_0805_2012Metric_Pad1.20x1.40mm_HandSolder"
 			(at 57.912 45.72 90)
 			(hide yes)
@@
 			)
 		)
-		(property "Footprint" ""
+		(property "Footprint" "Capacitor_SMD:C_0805_2012Metric_Pad1.18x1.45mm_HandSolder"
 			(at 68.2752 43.18 0)
 			(hide yes)
@@
 		(dnp no)
 		(property "Reference" "D1"
-			(at 56.388 22.352 0)
+			(at 55.626 22.352 0)
 			(show_name no)
 			(do_not_autoplace no)
@@
 			)
 		)
-		(property "Value" "D_Schottky"
-			(at 56.388 19.558 0)
+		(property "Value" "1N5819"
+			(at 55.626 24.638 0)
 			(show_name no)
 			(do_not_autoplace no)
@@
 			)
 		)
-		(property "Footprint" ""
+		(property "Footprint" "Diode_THT:D_DO-15_P12.70mm_Horizontal"
 			(at 55.88 27.94 0)
 			(hide yes)
@@
 			)
 		)
-		(property "Datasheet" ""
+		(property "Datasheet" "https://www.tme.eu/Document/7e78c56f041fe00f7158152d6ddb2c6e/1n5817.pdf"
 			(at 55.88 27.94 0)
 			(hide yes)
@@
 			)
 		)
+		(property "URL" "https://www.tme.eu/pl/details/1n5819-dio/diody-schottky-tht/diotec-semiconductor/1n5819/"
+			(at 55.88 27.94 0)
+			(hide yes)
+			(show_name no)
+			(do_not_autoplace no)
+			(effects
+				(font
+					(size 1.27 1.27)
+				)
+			)
+		)
+		(property "TME" "1N5819-DIO"
+			(at 55.88 27.94 0)
+			(hide yes)
+			(show_name no)
+			(do_not_autoplace no)
+			(effects
+				(font
+					(size 1.27 1.27)
+				)
+			)
+		)
+		(property "MAN" "1N5819"
+			(at 55.88 27.94 0)
+			(hide yes)
+			(show_name no)
+			(do_not_autoplace no)
+			(effects
+				(font
+					(size 1.27 1.27)
+				)
+			)
+		)
 		(pin "2"
 		)
@@
 			)
 		)
-		(property "Footprint" "Package_SO:SOIC-8_3.9x4.9mm_P1.27mm"
+		(property "Footprint" "Capacitor_SMD:C_0805_2012Metric_Pad1.18x1.45mm_HandSolder"
 			(at 45.4152 119.38 0)
 			(hide yes)

Commit message: usb finished
Parts:
- added C10: 100nF, Capacitor_SMD:C_0805_2012Metric_Pad1.18x1.45mm_HandSolder, symbol Device:C
- added C11, C12: 10uF, Capacitor_SMD:C_0805_2012Metric_Pad1.18x1.45mm_HandSolder, symbol Device:C
- added D2: 1N5908, Diode_THT:D_DO-201AE_P15.24mm_Horizontal, symbol Diode:1N62xxA
- added D3: LED_PWR, LED_THT:LED_D5.0mm, symbol Device:LED
- added R3: 1k, symbol Device:R
- added U2: LT1963AxST-1.5, Package_TO_SOT_SMD:SOT-223-3_TabPin2, symbol Regulator_Linear:LT1963AxST-1.5
Connections:
- net +3.3V: now also C12.1, R3.1, U2.3 (OUT)
- net +5V: now also C10.1, C11.1, D2.1 (A1), U2.1 (IN)
- net GND: now also C10.2, C11.2, C12.2, D2.2 (A2), D3.1 (K), U2.2 (GND)
- net PC13: now reaches U1.1 (PC13)
- net PA0: now reaches U1.11 (PA0)
- net PA1: now reaches U1.12 (PA1)
- net PA2: now reaches U1.13 (PA2)
- net PA3: now reaches U1.14 (PA3)
- net PA4: now reaches U1.15 (PA4)
- net PA5: now reaches U1.16 (PA5)
- net PA6: now reaches U1.17 (PA6)
- net PA7: now reaches U1.18 (PA7)
- net PB0: now reaches U1.19 (PB0)
- net PB1: now reaches U1.20 (PB1)
- net PB2: now reaches U1.21 (PB2)
- net PB10: now reaches U1.22 (PB10)
- net PB11: now reaches U1.23 (PB11)
- net PB12: now reaches U1.24 (PB12)
- net PB13: now reaches U1.25 (PB13)
- net PB14: now reaches U1.26 (PB14)
- net PB15: now reaches U1.27 (PB15)
- net PA8: now reaches U1.28 (PA8)
- net PC6: now reaches U1.30 (PC6)
- net PC7: now reaches U1.31 (PC7)
- net PA9: now reaches U1.33 (PA9/PA11)
- net PA10: now reaches U1.34 (PA10/PA12)
- net PA15: now reaches U1.37 (PA15)
- net PD0: now reaches U1.38 (PD0)
- net PD1: now reaches U1.39 (PD1)
- net PD2: now reaches U1.40 (PD2)
- net PD3: now reaches U1.41 (PD3)
- net PB3: now reaches U1.42 (PB3)
- net PB4: now reaches U1.43 (PB4)
- net PB5: now reaches U1.44 (PB5)
- net PB6: now reaches U1.45 (PB6)
- net PB7: now reaches U1.46 (PB7)
- net PB8: now reaches U1.47 (PB8)
- net PB9: now reaches U1.48 (PB9)
- new net: D3.2 (A), R3.2
Other:
- note added: "USB as a supply voltage"
- note added: "Voltage regulator for uC"
- moved on the sheet: C1, C2, C3, C4, C5, C6, C7, C8, C9, D1, J1, J2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

Commit message: Connectors
Parts:
- added C13: 10nF, Capacitor_SMD:C_0805_2012Metric_Pad1.18x1.45mm_HandSolder, symbol Device:C
- added D4: LED, LED_THT:LED_D5.0mm, symbol Device:LED
- added J3: East, symbol Connector_Generic:Conn_01x11
- added J4: South, symbol Connector_Generic:Conn_01x12
- added J5: North, Connector_PinHeader_2.54mm:PinHeader_1x12_P2.54mm_Vertical, symbol Connector_Generic:Conn_01x12
- added J6: West, symbol Connector_Generic:Conn_01x02
- added R4, R5: 1k, Resistor_SMD:R_0805_2012Metric_Pad1.20x1.40mm_HandSolder, symbol Device:R
- added R6: 10k, Resistor_SMD:R_0805_2012Metric_Pad1.20x1.40mm_HandSolder, symbol Device:R
- added SW2: RST, Button_Switch_THT:SW_PUSH_6mm_2pin, symbol Switch:SW_Push
- U2: value LT1963AxST-1.5 -> TPS1117LV33S
Connections:
- net +3.3V: now also R6.1
- net GND: now also C13.2, D4.1 (K), SW2.2
- net PA0: now also J6.2 (Pin_2)
- net PA1: now also J6.1 (Pin_1)
- net PA10: now also J3.4 (Pin_4)
- net PA15: now also J5.12 (Pin_12)
- net PA2: now also J4.12 (Pin_12)
- net PA3: now also J4.11 (Pin_11)
- net PA4: now also J4.10 (Pin_10)
- net PA5: now also J4.9 (Pin_9); no longer U1.16 (PA5)
- net PA6: now also J4.8 (Pin_8)
- net PA7: now also J4.7 (Pin_7)
- net PA8: now also J3.8 (Pin_8)
- net PA9: now also J3.7 (Pin_7)
- net PB0: now also J4.6 (Pin_6)
- net PB1: now also J4.5 (Pin_5)
- net PB10: now also J4.3 (Pin_3)
- net PB11: now also J4.2 (Pin_2)
- net PB12: now also J4.1 (Pin_1)
- net PB13: now also J3.11 (Pin_11)
- net PB14: now also J3.10 (Pin_10)
- net PB15: now also J3.9 (Pin_9)
- net PB2: now also J4.4 (Pin_4)
- net PB3: now also J5.7 (Pin_7)
- net PB4: now also J5.6 (Pin_6)
- net PB5: now also J5.5 (Pin_5)
- net PB6: now also J5.4 (Pin_4)
- net PB7: now also J5.3 (Pin_3)
- net PB8: now also J5.2 (Pin_2)
- net PB9: now also J5.1 (Pin_1)
- net PC6: now also J3.6 (Pin_6)
- net PC7: now also J3.5 (Pin_5)
- net PD0: now also J5.11 (Pin_11)
- net PD1: now also J5.10 (Pin_10)
- net PD2: now also J5.9 (Pin_9)
- net PD3: now also J5.8 (Pin_8)
- net PC13 renamed PC13-USR_BTN
- net PC13-USR_BTN: now also R5.1
- new net: C13.1, R5.2, R6.2, SW2.1
- new net: D4.2 (A), R4.2
- new net PA11: J3.3 (Pin_3)
- new net PA12: J3.2 (Pin_2)
- new net PA13: J3.1 (Pin_1)
- new net PA5-USR_LED: R4.1, U1.16 (PA5)
Other:
- note added: "Connectors"
- note added: "USR LED and BTN"
- moved on the sheet: C11, C12, C4, C5, C6, C7, C8, D3, J1, R3, SW1, U1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

Commit message: some changes in connectors
nothing special
Parts:
- removed J4: South, symbol Connector_Generic:Conn_01x12
- added J7: South, Connector_PinHeader_2.54mm:PinHeader_1x11_P2.54mm_Vertical, symbol Connector_Generic:Conn_01x11
- J1: footprint Package_DFN_QFN:QFN-24-1EP_4x4mm_P0.5mm_EP2.6x2.6mm -> Connector_PinHeader_2.54mm:PinHeader_1x05_P2.54mm_Vertical
- J3: footprint (none) -> Connector_PinHeader_2.54mm:PinHeader_1x11_P2.54mm_Vertical
- J6: footprint (none) -> Connector_PinHeader_2.54mm:PinHeader_1x02_P2.54mm_Vertical
Connections:
- net PA2: now also J7.11 (Pin_11)
- net PA3: now also J7.10 (Pin_10)
- net PA4: now also J7.9 (Pin_9)
- net PA6: now also J7.8 (Pin_8)
- net PA7: now also J7.7 (Pin_7)
- net PB0: now also J7.6 (Pin_6)
- net PB1: now also J7.5 (Pin_5)
- net PB10: now also J7.3 (Pin_3)
- net PB11: now also J7.2 (Pin_2)
- net PB12: now also J7.1 (Pin_1)
- net PB2: now also J7.4 (Pin_4)

Commit message: schematic main part done
Parts:
- removed J3: East, Connector_PinHeader_2.54mm:PinHeader_1x11_P2.54mm_Vertical, symbol Connector_Generic:Conn_01x11
- added J3: PA-PC-PB-Conn, symbol Connector_Generic:Conn_01x10
- J5: value North -> PB-PD-Conn
- J6: value West -> PA-Conn
- J7: value South -> PA-PB-Conn
- R3: footprint (none) -> Resistor_SMD:R_0805_2012Metric_Pad1.20x1.40mm_HandSolder
- SW2: value RST -> USR_BTN
Connections:
- net PA10: now also U1.32 (PA10), J3.3 (Pin_3); no longer U1.34 (PA10/PA12)
- net PA11: now also U1.33 (PA11), J3.2 (Pin_2)
- net PA12: now also U1.34 (PA12), J3.1 (Pin_1)
- net PA8: now also J3.7 (Pin_7)
- net PA9: now also U1.29 (PA9), J3.6 (Pin_6); no longer U1.33 (PA9/PA11)
- net PB13: now also J3.10 (Pin_10)
- net PB14: now also J3.9 (Pin_9)
- net PB15: now also J3.8 (Pin_8)
- net PC6: now also J3.5 (Pin_5)
- net PC7: now also J3.4 (Pin_4)

Commit message: pcb init and bill
Parts:
- J3: footprint (none) -> Connector_PinHeader_2.54mm:PinHeader_1x10_P2.54mm_Vertical
Changed lines of the file:
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@@
 			)
 		)
-		(property "Footprint" ""
+		(property "Footprint" "Connector_PinHeader_2.54mm:PinHeader_1x10_P2.54mm_Vertical"
 			(at 281.94 134.62 0)
 			(hide yes)
